File: Hardware/Pi_Block.sch (EAGLE design)
At the start: 53 parts, among them Q1 200mA/50V, U1 PCA9306, U2 EDISON_CONNECTOR_FULLMOUNTING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, U3 EDISON_CONNECTOR_FULLHEADER, U4 TPS62065, U5 MIC5219 3.3V, U6 TXB0108, U7 TXB0108

Commit message: Fixed silk on PCA. Added dimensions.
Other:
- moved on the sheet: Q1, R11, R9
Changed lines of the file:
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@@
 <instance part="GND25" gate="1" x="96.52" y="48.26"/>
 <instance part="S1" gate="G$1" x="96.52" y="167.64" rot="MR0"/>
-<instance part="R9" gate="G$1" x="91.44" y="177.8" smashed="yes" rot="R180">
-<attribute name="NAME" x="95.25" y="181.3814" size="1.778" layer="95" rot="R180"/>
-<attribute name="VALUE" x="95.25" y="176.022" size="1.778" layer="96" rot="R180"/>
+<instance part="R9" gate="G$1" x="93.98" y="177.8" smashed="yes" rot="R180">
+<attribute name="NAME" x="97.79" y="181.3814" size="1.778" layer="95" rot="R180"/>
+<attribute name="VALUE" x="97.79" y="176.022" size="1.778" layer="96" rot="R180"/>
 </instance>
 <instance part="R10" gate="G$1" x="78.74" y="167.64">
@@
 <instance part="GND26" gate="1" x="104.14" y="162.56"/>
 <instance part="LOGO3" gate="G$1" x="238.76" y="38.1"/>
-<instance part="Q1" gate="G$1" x="137.16" y="162.56"/>
-<instance part="R11" gate="G$1" x="124.46" y="162.56" rot="R180"/>
-<instance part="SUPPLY8" gate="G$1" x="116.84" y="165.1"/>
+<instance part="Q1" gate="G$1" x="132.08" y="157.48" smashed="yes">
+<attribute name="NAME" x="137.16" y="160.02" size="1.778" layer="95"/>
+<attribute name="VALUE" x="137.16" y="157.48" size="1.778" layer="96"/>
+</instance>
+<instance part="R11" gate="G$1" x="121.92" y="165.1" rot="R90"/>
+<instance part="SUPPLY8" gate="G$1" x="121.92" y="172.72"/>
 <instance part="D1" gate="G$1" x="139.7" y="114.3" smashed="yes" rot="R90">
 <attribute name="NAME" x="142.24" y="114.3" size="1.778" layer="95"/>
@@
 </segment>
 <segment>
-<wire x1="96.52" y1="177.8" x2="99.06" y2="177.8" width="0.1524" layer="91"/>
+<wire x1="99.06" y1="177.8" x2="101.6" y2="177.8" width="0.1524" layer="91"/>
 <pinref part="R9" gate="G$1" pin="1"/>
-<label x="99.06" y="177.8" size="1.778" layer="95" xref="yes"/>
+<label x="101.6" y="177.8" size="1.778" layer="95" xref="yes"/>
 </segment>
 <segment>
 <pinref part="Q1" gate="G$1" pin="D"/>
-<wire x1="137.16" y1="167.64" x2="137.16" y2="170.18" width="0.1524" layer="91"/>
-<wire x1="137.16" y1="170.18" x2="139.7" y2="170.18" width="0.1524" layer="91"/>
-<label x="139.7" y="170.18" size="1.27" layer="95" xref="yes"/>
+<wire x1="132.08" y1="162.56" x2="132.08" y2="165.1" width="0.1524" layer="91"/>
+<wire x1="132.08" y1="165.1" x2="139.7" y2="165.1" width="0.1524" layer="91"/>
+<label x="139.7" y="165.1" size="1.27" layer="95" xref="yes"/>
 </segment>
 <segment>
@@
 <pinref part="SUPPLY8" gate="G$1" pin="5V"/>
 <pinref part="R11" gate="G$1" pin="2"/>
-<wire x1="116.84" y1="165.1" x2="116.84" y2="162.56" width="0.1524" layer="91"/>
-<wire x1="116.84" y1="162.56" x2="119.38" y2="162.56" width="0.1524" layer="91"/>
+<wire x1="121.92" y1="172.72" x2="121.92" y2="170.18" width="0.1524" layer="91"/>
 </segment>
 <segment>
@@
 <wire x1="83.82" y1="167.64" x2="86.36" y2="167.64" width="0.1524" layer="91"/>
 <wire x1="86.36" y1="167.64" x2="86.36" y2="177.8" width="0.1524" layer="91"/>
+<wire x1="86.36" y1="177.8" x2="88.9" y2="177.8" width="0.1524" layer="91"/>
 <junction x="86.36" y="167.64"/>
 <pinref part="S1" gate="G$1" pin="2"/>
@@
 <net name="DCIN" class="0">
 <segment>
-<wire x1="137.16" y1="154.94" x2="139.7" y2="154.94" width="0.1524" layer="91"/>
-<label x="139.7" y="154.94" size="1.27" layer="95" xref="yes"/>
+<wire x1="132.08" y1="149.86" x2="139.7" y2="149.86" width="0.1524" layer="91"/>
+<label x="139.7" y="149.86" size="1.27" layer="95" xref="yes"/>
 <pinref part="Q1" gate="G$1" pin="S"/>
-<wire x1="137.16" y1="154.94" x2="137.16" y2="157.48" width="0.1524" layer="91"/>
+<wire x1="132.08" y1="149.86" x2="132.08" y2="152.4" width="0.1524" layer="91"/>
 </segment>
 </net>
@@
 <pinref part="Q1" gate="G$1" pin="G"/>
 <pinref part="R11" gate="G$1" pin="1"/>
-</segment>
-</net>
+<wire x1="124.46" y1="157.48" x2="121.92" y2="157.48" width="0.1524" layer="91"/>
+<wire x1="121.92" y1="157.48" x2="121.92" y2="160.02" width="0.1524" layer="91"/>
+</segment>
+</net>
